Commit message: porting to melodic

File: katana_description/urdf/controlbox.urdf.xacro (robot description, xacro)
@@ -1,6 +1,6 @@
 <?xml version="1.0"?>
 <robot xmlns:xacro="http://ros.org/wiki/xacro" >
-  <property name="M_PI" value="3.1415926535897931" />
-  <property name="controlbox_height" value="0.073" />
+  <xacro:property name="M_PI" value="3.1415926535897931" />
+  <xacro:property name="controlbox_height" value="0.073" />
   <link name="katana_internal_controlbox_link">
     <visual>

File: katana_description/urdf/katana_300_6m180.urdf.xacro (robot description, xacro)
@@ -4,11 +4,11 @@
   <xacro:include filename="$(find katana_description)/urdf/transmissions.urdf.xacro"/>
   <xacro:include filename="$(find katana_description)/urdf/gazebo.urdf.xacro"/>
-  <property name="M_PI" value="3.1415926535897931" />
+  <xacro:property name="M_PI" value="3.1415926535897931" />
   <!-- all values from the katana manual -->
-  <property name="base_height" value="0.2015" />
-  <property name="link2_length" value="0.19" />
-  <property name="link3_length" value="0.139" />
-  <property name="link4_length" value="0.1523" />
-  <property name="link5_length" value="0.1505" />
+  <xacro:property name="base_height" value="0.2015" />
+  <xacro:property name="link2_length" value="0.19" />
+  <xacro:property name="link3_length" value="0.139" />
+  <xacro:property name="link4_length" value="0.1523" />
+  <xacro:property name="link5_length" value="0.1505" />
   <!-- All inertial values (mass, center of mass and inertia tensor) have been
        calculated from the meshes using MeshLab -->

File: katana_description/urdf/katana_400_6m180.urdf.xacro (robot description, xacro)
@@ -4,11 +4,11 @@
   <xacro:include filename="$(find katana_description)/urdf/transmissions.urdf.xacro"/>
   <xacro:include filename="$(find katana_description)/urdf/gazebo.urdf.xacro"/>
-  <property name="M_PI" value="3.1415926535897931" />
+  <xacro:property name="M_PI" value="3.1415926535897931" />
   <!-- all values from the katana manual -->
-  <property name="base_height" value="0.2015" />
-  <property name="link2_length" value="0.19" />
-  <property name="link3_length" value="0.139" />
-  <property name="link4_length" value="0.1523" />
-  <property name="link5_length" value="0.1505" />
+  <xacro:property name="base_height" value="0.2015" />
+  <xacro:property name="link2_length" value="0.19" />
+  <xacro:property name="link3_length" value="0.139" />
+  <xacro:property name="link4_length" value="0.1523" />
+  <xacro:property name="link5_length" value="0.1505" />
   <!-- All inertial values (mass, center of mass and inertia tensor) have been
        calculated from the meshes using MeshLab -->

File: katana_description/urdf/katana_450_6m90a.urdf.xacro (robot description, xacro)
@@ -4,12 +4,12 @@
   <xacro:include filename="$(find katana_description)/urdf/transmissions.urdf.xacro"/>
   <xacro:include filename="$(find katana_description)/urdf/gazebo.urdf.xacro"/>
-  <property name="M_PI" value="3.1415926535897931" />
+  <xacro:property name="M_PI" value="3.1415926535897931" />
   <!-- all values from the katana manual -->
-  <property name="base_height" value="0.2015" />
-  <property name="link2_length" value="0.19" />
-  <property name="link3_length" value="0.139" />
-  <property name="link4_length" value="0.1473" />
-  <property name="link5_length" value="0.1505" />
-  <property name="tool_frame_offset" value="0.11" />
+  <xacro:property name="base_height" value="0.2015" />
+  <xacro:property name="link2_length" value="0.19" />
+  <xacro:property name="link3_length" value="0.139" />
+  <xacro:property name="link4_length" value="0.1473" />
+  <xacro:property name="link5_length" value="0.1505" />
+  <xacro:property name="tool_frame_offset" value="0.11" />
   <!-- All inertial values (mass, center of mass and inertia tensor) have been
        calculated from the meshes using MeshLab -->
@@ -260,5 +260,5 @@
         <inertial>
           <mass value="0.0251722230462" />
-          <origin xyz="${0.034 + (-0.032216)} 0.025167 -.001603"/>
+          <origin xyz="${0.034 + (-0.032216)} 0.025167 -0.001603"/>
           <inertia ixx="0.000005990" ixy="0.000008473" ixz="0.000001448"
             iyy="0.000019757" iyz="-0.000000996"

File: katana_description/urdf/katana_450_6m90b.urdf.xacro (robot description, xacro)
@@ -4,11 +4,11 @@
   <xacro:include filename="$(find katana_description)/urdf/transmissions.urdf.xacro"/>
   <xacro:include filename="$(find katana_description)/urdf/gazebo.urdf.xacro"/>
-  <property name="M_PI" value="3.1415926535897931" />
+  <xacro:property name="M_PI" value="3.1415926535897931" />
   <!-- all values from the katana manual -->
-  <property name="base_height" value="0.2015" />
-  <property name="link2_length" value="0.19" />
-  <property name="link3_length" value="0.139" />
-  <property name="link4_length" value="0.1473" />
-  <property name="link5_length" value="0.1505" />
+  <xacro:property name="base_height" value="0.2015" />
+  <xacro:property name="link2_length" value="0.19" />
+  <xacro:property name="link3_length" value="0.139" />
+  <xacro:property name="link4_length" value="0.1473" />
+  <xacro:property name="link5_length" value="0.1505" />
   <!-- All inertial values (mass, center of mass and inertia tensor) have been
        calculated from the meshes using MeshLab -->

File: katana_description/urdf/transmissions.urdf.xacro (robot description, xacro)
@@ -6,5 +6,5 @@
       <type>transmission_interface/SimpleTransmission</type>
       <joint name="${name}_joint">
-        <hardwareInterface>EffortJointInterface</hardwareInterface>
+        <hardwareInterface>hardware_interface/EffortJointInterface</hardwareInterface>
       </joint>
       <actuator name="${name}_motor">
